File: pathfinderKey-Cuts.kicad_pcb (KiCad board)
At the start: 2 copper layers, 81 x 71 mm, 13 parts, among them SW1 SW_Push, SW2 SW_Push, SW3 SW_Push, SW4 SW_Push, U1 XIAO-RP2040-DIP

Commit message: Add files via upload
Routing:
- net button1: track 116.0 -> 111.4 mm
Changed lines of the file:
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@@
-	)
-	(segment
-		(start 145.288 112.268)
-		(end 151.5 112.268)
-		(width 0.2)
-		(layer "B.Cu")
-		(net 8)
 	)
 	(segment
@@
 	)
 	(segment
-		(start 124.12 122.88)
-		(end 124 123)
+		(start 145.288 101.892)
+		(end 151.5 95.68)
+		(width 0.2)
+		(layer "B.Cu")
+		(net 8)
+	)
+	(segment
+		(start 166 91.5)
+		(end 182.62 91.5)
+		(width 0.2)
+		(layer "B.Cu")
+		(net 8)
+	)
+	(segment
+		(start 142.556 115)
+		(end 145.288 112.268)
 		(width 0.2)
 		(layer "B.Cu")
@@
 	)
 	(segment
-		(start 124 123)
+		(start 153.77 80.23)
+		(end 162.23 80.23)
+		(width 0.2)
+		(layer "B.Cu")
+		(net 8)
+	)
+	(segment
+		(start 127 115)
+		(end 142.556 115)
+		(width 0.2)
+		(layer "B.Cu")
+		(net 8)
+	)
+	(segment
+		(start 182.62 91.5)
+		(end 187.54 96.42)
+		(width 0.2)
+		(layer "B.Cu")
+		(net 8)
+	)
+	(segment
+		(start 151.5 95.68)
+		(end 151.5 82.5)
+		(width 0.2)
+		(layer "B.Cu")
+		(net 8)
+	)
+	(segment
+		(start 124 121.43)
 		(end 124 118)
 		(width 0.2)
@@
 	)
 	(segment
-		(start 127.26 122.88)
-		(end 124.12 122.88)
+		(start 125.53 122.88)
+		(end 125.49 122.92)
 		(width 0.2)
 		(layer "B.Cu")
@@
 	)
 	(segment
-		(start 151.5 112.268)
-		(end 151.5 82.5)
+		(start 125.49 122.92)
+		(end 124 121.43)
 		(width 0.2)
 		(layer "B.Cu")
@@
 	)
 	(segment
-		(start 153.77 80.23)
-		(end 162.23 80.23)
-		(width 0.2)
-		(layer "B.Cu")
-		(net 8)
-	)
-	(segment
-		(start 182.62 91.5)
-		(end 187.54 96.42)
+		(start 145.288 112.268)
+		(end 145.288 101.892)
 		(width 0.2)
 		(layer "B.Cu")
@@
 	)
 	(segment
-		(start 166 91.5)
-		(end 182.62 91.5)
-		(width 0.2)
-		(layer "B.Cu")
-		(net 8)
-	)
-	(segment
-		(start 127 115)
-		(end 142.556 115)
+		(start 127.26 122.88)
+		(end 125.53 122.88)
 		(width 0.2)
 		(layer "B.Cu")
@@
 	)
 	(segment
-		(start 142.556 115)
-		(end 145.288 112.268)
+		(start 150.112 119.888)
+		(end 145.288 119.888)
 		(width 0.2)
 		(layer "B.Cu")
-		(net 8)
+		(net 9)
 	)
 	(segment
-		(start 129.5 118.5)
-		(end 129.5 123.18)
+		(start 156 114)
+		(end 150.112 119.888)
+		(width 0.2)
+		(layer "B.Cu")
+		(net 9)
+	)
+	(segment
+		(start 163.369 96.42)
+		(end 162.58 96.42)
+		(width 0.2)
+		(layer "B.Cu")
+		(net 9)
+	)
+	(segment
+		(start 130 118)
+		(end 129.5 118.5)
 		(width 0.2)
 		(layer "B.Cu")
@@
 	)
 	(segment
-		(start 156 103)
-		(end 156 114)
+		(start 145.288 119.888)
+		(end 143.4 118)
 		(width 0.2)
 		(layer "B.Cu")
@@
 	)
 	(segment
-		(start 163.369 96.42)
-		(end 162.58 96.42)
-		(width 0.2)
-		(layer "B.Cu")
-		(net 9)
-	)
-	(segment
-		(start 149.86 119.888)
-		(end 151.748 118)
-		(width 0.2)
-		(layer "B.Cu")
-		(net 9)
-	)
-	(segment
-		(start 151.748 118)
-		(end 152 118)
-		(width 0.2)
-		(layer "B.Cu")
-		(net 9)
-	)
-	(segment
-		(start 145.288 119.888)
-		(end 149.86 119.888)
-		(width 0.2)
-		(layer "B.Cu")
-		(net 9)
-	)
-	(segment
-		(start 130 118)
-		(end 129.5 118.5)
-		(width 0.2)
-		(layer "B.Cu")
-		(net 9)
-	)
-	(segment
-		(start 156 114)
-		(end 152 118)
+		(start 129.5 118.5)
+		(end 129.5 123.18)
 		(width 0.2)
 		(layer "B.Cu")
@@
 	)
 	(segment
-		(start 130 118)
-		(end 143.4 118)
+		(start 143.4 118)
+		(end 130 118)
 		(width 0.2)
 		(layer "B.Cu")
@@
 	)
 	(segment
-		(start 143.4 118)
-		(end 145.288 119.888)
+		(start 156 103)
+		(end 156 114)
 		(width 0.2)
 		(layer "B.Cu")
